File: Adafruit NeoPixel 8 Stick v2.brd (EAGLE design)
At the start: 50.8 x 10.2 mm, 24 parts, among them CN1 1X4SMT, CN2 1X4SMT

Commit message: Fixed consistency board<>schematic
Parts:
- LED1, LED2, LED3, LED4, LED5, LED6, LED7, LED8: value WS2812B5050 -> WS2812B5050-NARROW
Changed lines of the file:
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@@
 <?xml version="1.0" encoding="utf-8"?>
 <!DOCTYPE eagle SYSTEM "eagle.dtd">
-<eagle version="6.3">
+<eagle version="9.6.2">
 <drawing>
 <settings>
 <setting alwaysvectorfont="no"/>
+<setting keepoldvectorfont="yes"/>
 <setting verticaltext="up"/>
 </settings>
@@
 <param name="dpMaxLengthDifference" value="10mm"/>
 <param name="dpGapFactor" value="2.5"/>
-<param name="checkGrid" value="0"/>
 <param name="checkAngle" value="1"/>
 <param name="checkFont" value="1"/>
 <param name="checkRestrict" value="1"/>
+<param name="checkStop" value="0"/>
+<param name="checkValues" value="0"/>
+<param name="checkNames" value="1"/>
+<param name="checkWireStubs" value="1"/>
+<param name="checkPolygonWidth" value="0"/>
 <param name="useDiameter" value="13"/>
 <param name="maxErrors" value="50"/>
@@
 <pass name="Default">
 <param name="RoutingGrid" value="50mil"/>
+<param name="AutoGrid" value="1"/>
+<param name="Efforts" value="0"/>
+<param name="TopRouterVariant" value="1"/>
 <param name="tpViaShape" value="round"/>
 <param name="PrefDir.1" value="|"/>
@@
 </autorouter>
 <elements>
-<element name="LED1" library="microbuilder" package="WS2812B-NARROW" value="WS2812B5050" x="3.175" y="3.81"/>
-<element name="LED2" library="microbuilder" package="WS2812B-NARROW" value="WS2812B5050" x="9.525" y="3.81"/>
-<element name="LED3" library="microbuilder" package="WS2812B-NARROW" value="WS2812B5050" x="15.875" y="3.81"/>
-<element name="LED4" library="microbuilder" package="WS2812B-NARROW" value="WS2812B5050" x="22.225" y="3.81"/>
-<element name="LED5" library="microbuilder" package="WS2812B-NARROW" value="WS2812B5050" x="28.575" y="3.81"/>
-<element name="LED6" library="microbuilder" package="WS2812B-NARROW" value="WS2812B5050" x="34.925" y="3.81"/>
-<element name="LED7" library="microbuilder" package="WS2812B-NARROW" value="WS2812B5050" x="41.275" y="3.81"/>
-<element name="LED8" library="microbuilder" package="WS2812B-NARROW" value="WS2812B5050" x="47.625" y="3.81"/>
-<element name="C1" library="rcl" package="C0805K" value="" x="8.382" y="8.382" rot="R180"/>
-<element name="C2" library="rcl" package="C0805K" value="" x="16.891" y="8.382" rot="R180"/>
-<element name="C3" library="rcl" package="C0805K" value="" x="22.225" y="8.382" rot="R180"/>
-<element name="C4" library="rcl" package="C0805K" value="" x="28.575" y="8.382" rot="R180"/>
-<element name="C5" library="rcl" package="C0805K" value="" x="33.655" y="8.382" rot="R180"/>
-<element name="C6" library="rcl" package="C0805K" value="" x="42.037" y="8.382" rot="R180"/>
-<element name="C7" library="rcl" package="C0805K" value="" x="48.26" y="8.382" rot="R180"/>
-<element name="FID1" library="microbuilder" package="FIDUCIAL_1MM" value="FIDUCIAL&quot;&quot;" x="5.334" y="8.382">
+<element name="LED1" library="microbuilder" package="WS2812B-NARROW" value="WS2812B5050-NARROW" x="3.175" y="3.81" smashed="yes">
+<attribute name="NAME" x="6.6675" y="5.3975" size="0.8128" layer="25" ratio="10" rot="R270"/>
+</element>
+<element name="LED2" library="microbuilder" package="WS2812B-NARROW" value="WS2812B5050-NARROW" x="9.525" y="3.81" smashed="yes">
+<attribute name="NAME" x="13.0175" y="5.3975" size="0.8128" layer="25" ratio="10" rot="R270"/>
+</element>
+<element name="LED3" library="microbuilder" package="WS2812B-NARROW" value="WS2812B5050-NARROW" x="15.875" y="3.81" smashed="yes">
+<attribute name="NAME" x="19.3675" y="5.3975" size="0.8128" layer="25" ratio="10" rot="R270"/>
+</element>
+<element name="LED4" library="microbuilder" package="WS2812B-NARROW" value="WS2812B5050-NARROW" x="22.225" y="3.81" smashed="yes">
+<attribute name="NAME" x="25.7175" y="5.3975" size="0.8128" layer="25" ratio="10" rot="R270"/>
+</element>
+<element name="LED5" library="microbuilder" package="WS2812B-NARROW" value="WS2812B5050-NARROW" x="28.575" y="3.81" smashed="yes">
+<attribute name="NAME" x="32.0675" y="5.3975" size="0.8128" layer="25" ratio="10" rot="R270"/>
+</element>
+<element name="LED6" library="microbuilder" package="WS2812B-NARROW" value="WS2812B5050-NARROW" x="34.925" y="3.81" smashed="yes">
+<attribute name="NAME" x="38.4175" y="5.3975" size="0.8128" layer="25" ratio="10" rot="R270"/>
+</element>
+<element name="LED7" library="microbuilder" package="WS2812B-NARROW" value="WS2812B5050-NARROW" x="41.275" y="3.81" smashed="yes">
+<attribute name="NAME" x="44.7675" y="5.3975" size="0.8128" layer="25" ratio="10" rot="R270"/>
+</element>
+<element name="LED8" library="microbuilder" package="WS2812B-NARROW" value="WS2812B5050-NARROW" x="47.625" y="3.81" smashed="yes">
+<attribute name="NAME" x="51.1175" y="5.3975" size="0.8128" layer="25" ratio="10" rot="R270"/>
+</element>
+<element name="C1" library="rcl" package="C0805K" value="" x="8.382" y="8.382" smashed="yes" rot="R180">
+<attribute name="NAME" x="9.382" y="7.507" size="1.016" layer="25" rot="R180"/>
+<attribute name="VALUE" x="9.382" y="10.282" size="1.016" layer="27" rot="R180"/>
+</element>
+<element name="C2" library="rcl" package="C0805K" value="" x="16.891" y="8.382" smashed="yes" rot="R180">
+<attribute name="NAME" x="17.891" y="7.507" size="1.016" layer="25" rot="R180"/>
+<attribute name="VALUE" x="17.891" y="10.282" size="1.016" layer="27" rot="R180"/>
+</element>
+<element name="C3" library="rcl" package="C0805K" value="" x="22.225" y="8.382" smashed="yes" rot="R180">
+<attribute name="NAME" x="23.225" y="7.507" size="1.016" layer="25" rot="R180"/>
+<attribute name="VALUE" x="23.225" y="10.282" size="1.016" layer="27" rot="R180"/>
+</element>
+<element name="C4" library="rcl" package="C0805K" value="" x="28.575" y="8.382" smashed="yes" rot="R180">
+<attribute name="NAME" x="29.575" y="7.507" size="1.016" layer="25" rot="R180"/>
+<attribute name="VALUE" x="29.575" y="10.282" size="1.016" layer="27" rot="R180"/>
+</element>
+<element name="C5" library="rcl" package="C0805K" value="" x="33.655" y="8.382" smashed="yes" rot="R180">
+<attribute name="NAME" x="34.655" y="7.507" size="1.016" layer="25" rot="R180"/>
+<attribute name="VALUE" x="34.655" y="10.282" size="1.016" layer="27" rot="R180"/>
+</element>
+<element name="C6" library="rcl" package="C0805K" value="" x="42.037" y="8.382" smashed="yes" rot="R180">
+<attribute name="NAME" x="43.037" y="7.507" size="1.016" layer="25" rot="R180"/>
+<attribute name="VALUE" x="43.037" y="10.282" size="1.016" layer="27" rot="R180"/>
+</element>
+<element name="C7" library="rcl" package="C0805K" value="" x="48.26" y="8.382" smashed="yes" rot="R180">
+<attribute name="NAME" x="49.26" y="7.507" size="1.016" layer="25" rot="R180"/>
+<attribute name="VALUE" x="49.26" y="10.282" size="1.016" layer="27" rot="R180"/>
+</element>
+<element name="FID1" library="microbuilder" package="FIDUCIAL_1MM" value="FIDUCIAL&quot;&quot;" x="5.334" y="8.382" smashed="yes">
 <attribute name="BOM" value="EXCLUDE" x="5.334" y="8.382" size="1.27" layer="27" font="vector" ratio="10" display="off"/>
 </element>
-<element name="FID3" library="microbuilder" package="FIDUCIAL_1MM" value="FIDUCIAL&quot;&quot;" x="45.085" y="8.382">
+<element name="FID3" library="microbuilder" package="FIDUCIAL_1MM" value="FIDUCIAL&quot;&quot;" x="45.085" y="8.382" smashed="yes">
 <attribute name="BOM" value="EXCLUDE" x="45.085" y="8.382" size="1.27" layer="27" font="vector" ratio="10" display="off"/>
 </element>
-<element name="CN1" library="adafruit" package="1X4-SMT" value="1X4SMT" x="49.403" y="5.08" rot="MR270"/>
-<element name="CN2" library="adafruit" package="1X4-SMT" value="1X4SMT" x="1.397" y="5.08" rot="MR90"/>
-<element name="U$2" library="microbuilder" package="MOUNTINGHOLE_2.0_PLATED" value="MOUNTINGHOLE2.0" x="12.7" y="8.128"/>
-<element name="U$3" library="microbuilder" package="MOUNTINGHOLE_2.0_PLATED" value="MOUNTINGHOLE2.0" x="38.1" y="8.128"/>
-<element name="U$4" library="microbuilder" package="ADAFRUIT_2.5MM" value="" x="24.257" y="7.493"/>
-<element name="U$1" library="microbuilder" package="ADAFRUIT_TEXT_20MM" value="" x="35.179" y="0.381" rot="MR0"/>
+<element name="CN1" library="adafruit" package="1X4-SMT" value="1X4SMT" x="49.403" y="5.08" smashed="yes" rot="MR270"/>
+<element name="CN2" library="adafruit" package="1X4-SMT" value="1X4SMT" x="1.397" y="5.08" smashed="yes" rot="MR90"/>
+<element name="U$2" library="microbuilder" package="MOUNTINGHOLE_2.0_PLATED" value="MOUNTINGHOLE2.0" x="12.7" y="8.128" smashed="yes"/>
+<element name="U$3" library="microbuilder" package="MOUNTINGHOLE_2.0_PLATED" value="MOUNTINGHOLE2.0" x="38.1" y="8.128" smashed="yes"/>
+<element name="U$4" library="microbuilder" package="ADAFRUIT_2.5MM" value="" x="24.257" y="7.493" smashed="yes"/>
+<element name="U$1" library="microbuilder" package="ADAFRUIT_TEXT_20MM" value="" x="35.179" y="0.381" smashed="yes" rot="MR0"/>
 <element name="R1" library="microbuilder" package="_0805MP" value="470 OHM," x="2.413" y="8.382" smashed="yes">
 <attribute name="NAME" x="0.8255" y="9.3345" size="0.8128" layer="25" ratio="18"/>
@@
 </signal>
 </signals>
+<mfgpreviewcolors>
+<mfgpreviewcolor name="soldermaskcolor" color="0xC8008000"/>
+<mfgpreviewcolor name="silkscreencolor" color="0xFFFEFEFE"/>
+<mfgpreviewcolor name="backgroundcolor" color="0xFF282828"/>
+<mfgpreviewcolor name="coppercolor" color="0xFFFFBF00"/>
+<mfgpreviewcolor name="substratecolor" color="0xFF786E46"/>
+</mfgpreviewcolors>
 </board>
 </drawing>
