File: Adafruit NeoPixel 8 Stick v2.sch (EAGLE design)
At the start: 22 parts, among them CN1 1X4SMT, CN2 1X4SMT

Commit message: Fixed consistency board<>schematic
Parts:
- LED1, LED2, LED3, LED4, LED5, LED6, LED7, LED8: value WS2812B5050 -> WS2812B5050-NARROW; device microbuilder:WS2812B5050 -> microbuilder:WS2812B5050-NARROW
